File: KIS-3R33S_breakout.kicad_pcb (KiCad board)
At the start: 2 copper layers, 57.4 x 21.6 mm, 16 parts, among them P1 Screw terminal, P2 Screw terminal, U1 KIS-3R33S_modif

Commit message: Tweaked SMD capacitor footprint (added thermal vias / TH pads).
Parts:
- moved LOGO1 19.4 mm to (164.0, 100.0)
- moved LOGO2 9.03 mm to (138.0, 100.0)
- moved G*** 7.00 mm to (150.5, 97.8)
Other:
- board text added: "KIS-3R33S_breakout V0.12.e 2015 - blog.spitzenpfeil.org"
- board text removed: "KIS-3R33S_breakout V0.12.d 2015 - blog.spitzenpfeil.org"
Changed lines of the file:
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@@
-(kicad_pcb (version 4) (host pcbnew "(2015-04-23 BZR 5622)-product")
+(kicad_pcb (version 4) (host pcbnew "(2015-07-20 BZR 5967, Git 8482637)-product")
   (general
     (links 25)
     (no_connects 0)
-    (area 126.607142 87.275 195.802403 115.000001)
+    (area 128.349999 89.149999 185.850001 110.850001)
     (thickness 1.6)
     (drawings 17)
@@
     (add_net GND)
   )
+  (module Capacitors:c_elec_SMD_12.5x13.5 (layer F.Cu)
+    (at 170.15 102.7 90)
+    (descr "SMT capacitor, aluminium electrolytic, 12.5x13.5")
+    (fp_text reference C1 (at 0 -8 90) (layer F.SilkS) hide
+      (effects (font (size 1 1) (thickness 0.2)))
+    )
+    (fp_text value "1mF, 25V" (at 0 8 90) (layer F.Fab)
+      (effects (font (size 1 1) (thickness 0.2)))
+    )
+    (fp_text user - (at -3.5 -3.5 90) (layer F.SilkS)
+      (effects (font (size 1.5 1.5) (thickness 0.2)))
+    )
+    (fp_text user + (at 3.5 -3.5 90) (layer F.SilkS)
+      (effects (font (size 1.5 1.5) (thickness 0.2)))
+    )
+    (fp_line (start 3.95 -6.75) (end 6.75 -3.95) (layer F.SilkS) (width 0.2))
+    (fp_line (start 6.75 3.95) (end 3.95 6.75) (layer F.SilkS) (width 0.2))
+    (fp_line (start -6.15 1.1) (end -6.15 -1.1) (layer F.SilkS) (width 0.2))
+    (fp_line (start -6.1 1.35) (end -6.1 -1.35) (layer F.SilkS) (width 0.2))
+    (fp_line (start -6 -1.7) (end -6 1.7) (layer F.SilkS) (width 0.2))
+    (fp_line (start -5.9 2.05) (end -5.9 -2.05) (layer F.SilkS) (width 0.2))
+    (fp_line (start -5.8 -2.3) (end -5.8 2.3) (layer F.SilkS) (width 0.2))
+    (fp_line (start -5.7 2.55) (end -5.7 -2.55) (layer F.SilkS) (width 0.2))
+    (fp_line (start -5.6 2.75) (end -5.6 -2.75) (layer F.SilkS) (width 0.2))
+    (fp_line (start -5.5 -2.95) (end -5.5 2.95) (layer F.SilkS) (width 0.2))
+    (fp_line (start -5.4 3.1) (end -5.4 -3.1) (layer F.SilkS) (width 0.2))
+    (fp_line (start -5.3 -3.3) (end -5.3 3.3) (layer F.SilkS) (width 0.2))
+    (fp_line (start -5.2 -3.45) (end -5.2 3.45) (layer F.SilkS) (width 0.2))
+    (fp_line (start -5.1 -3.6) (end -5.1 3.6) (layer F.SilkS) (width 0.2))
+    (fp_line (start -2.2 -0.45) (end -7.45 -0.45) (layer Dwgs.User) (width 0.2))
+    (fp_line (start -2.2 0.45) (end -2.2 -0.45) (layer Dwgs.User) (width 0.2))
+    (fp_line (start -7.45 0.45) (end -2.2 0.45) (layer Dwgs.User) (width 0.2))
+    (fp_line (start -7.45 -0.45) (end -7.45 0.45) (layer Dwgs.User) (width 0.2))
+    (fp_line (start 2.2 0.45) (end 2.2 -0.45) (layer Dwgs.User) (width 0.2))
+    (fp_line (start 7.45 0.45) (end 2.2 0.45) (layer Dwgs.User) (width 0.2))
+    (fp_line (start 7.45 -0.45) (end 7.45 0.45) (layer Dwgs.User) (width 0.2))
+    (fp_line (start 2.2 -0.45) (end 7.45 -0.45) (layer Dwgs.User) (width 0.2))
+    (fp_line (start -6.75 6.75) (end -6.75 -6.75) (layer F.SilkS) (width 0.2))
+    (fp_line (start 3.95 6.75) (end -6.75 6.75) (layer F.SilkS) (width 0.2))
+    (fp_line (start 6.75 -3.95) (end 6.75 3.95) (layer F.SilkS) (width 0.2))
+    (fp_line (start -6.75 -6.75) (end 3.95 -6.75) (layer F.SilkS) (width 0.2))
+    (fp_circle (center 0 0) (end 6.25 0) (layer F.SilkS) (width 0.2))
+    (pad 1 smd rect (at 4.7 0 90) (size 6.3 2.5) (layers F.Cu F.Paste F.Mask)
+      (net 1 /Vout))
+    (pad 2 smd rect (at -4.7 0 90) (size 6.3 2.5) (layers F.Cu F.Paste F.Mask)
+      (net 4 GND))
+    (pad 1 thru_hole rect (at 2.54 0 90) (size 2.5 2.5) (drill 0.75) (layers *.Cu *.Mask)
+      (net 1 /Vout))
+    (pad 2 thru_hole rect (at -2.54 0 90) (size 2.5 2.5) (drill 0.75) (layers *.Cu *.Mask)
+      (net 4 GND))
+    (pad 1 thru_hole rect (at 3.81 0 90) (size 3 2.5) (drill 0.75) (layers *.Cu *.Mask)
+      (net 1 /Vout))
+    (pad 1 thru_hole rect (at -3.81 0 90) (size 3 2.5) (drill 0.75) (layers *.Cu *.Mask)
+      (net 1 /Vout))
+  )
   (module LOGO (layer B.Cu)
-    (at 157.5 97.8 180)
+    (at 150.5 97.8 180)
     (fp_text reference G*** (at 0 0 180) (layer B.SilkS) hide
       (effects (font (thickness 0.3)) (justify mirror))
@@
   )
   (module led-smile:LED_smile_silkscreen_6mm (layer B.Cu)
-    (at 182.1 107 180)
+    (at 164 100 180)
     (fp_text reference LOGO1 (at 0 -3.45694 180) (layer B.SilkS) hide
       (effects (font (size 0.127 0.127) (thickness 0.01524)) (justify mirror))
@@
   )
   (module oshw-logo:OSHW-logo_silkscreen_6mm (layer B.Cu)
-    (at 132.3 107 180)
+    (at 138 100 180)
     (fp_text reference LOGO2 (at 0 -3.18008 180) (layer B.SilkS) hide
       (effects (font (size 0.27178 0.27178) (thickness 0.05334)) (justify mirror))
@@
     )
   )
-  (module Capacitors:c_elec_SMD_12.5x13.5 (layer F.Cu)
-    (at 170.15 102.7 90)
-    (descr "SMT capacitor, aluminium electrolytic, 12.5x13.5")
-    (fp_text reference C1 (at 0 -8 90) (layer F.SilkS) hide
-      (effects (font (size 1 1) (thickness 0.15)))
-    )
-    (fp_text value "1mF, 25V" (at 0 8 90) (layer F.Fab)
-      (effects (font (size 1 1) (thickness 0.15)))
-    )
-    (fp_text user - (at -3.5 -3.5 90) (layer F.SilkS)
-      (effects (font (size 1.5 1.5) (thickness 0.15)))
-    )
-    (fp_text user + (at 3.5 -3.5 90) (layer F.SilkS)
-      (effects (font (size 1.5 1.5) (thickness 0.15)))
-    )
-    (fp_line (start 3.95 -6.75) (end 6.75 -3.95) (layer F.SilkS) (width 0.15))
-    (fp_line (start 6.75 3.95) (end 3.95 6.75) (layer F.SilkS) (width 0.15))
-    (fp_line (start -6.15 1.1) (end -6.15 -1.1) (layer F.SilkS) (width 0.15))
-    (fp_line (start -6.1 1.35) (end -6.1 -1.35) (layer F.SilkS) (width 0.15))
-    (fp_line (start -6 -1.7) (end -6 1.7) (layer F.SilkS) (width 0.15))
-    (fp_line (start -5.9 2.05) (end -5.9 -2.05) (layer F.SilkS) (width 0.15))
-    (fp_line (start -5.8 -2.3) (end -5.8 2.3) (layer F.SilkS) (width 0.15))
-    (fp_line (start -5.7 2.55) (end -5.7 -2.55) (layer F.SilkS) (width 0.15))
-    (fp_line (start -5.6 2.75) (end -5.6 -2.75) (layer F.SilkS) (width 0.15))
-    (fp_line (start -5.5 -2.95) (end -5.5 2.95) (layer F.SilkS) (width 0.15))
-    (fp_line (start -5.4 3.1) (end -5.4 -3.1) (layer F.SilkS) (width 0.15))
-    (fp_line (start -5.3 -3.3) (end -5.3 3.3) (layer F.SilkS) (width 0.15))
-    (fp_line (start -5.2 -3.45) (end -5.2 3.45) (layer F.SilkS) (width 0.15))
-    (fp_line (start -5.1 -3.6) (end -5.1 3.6) (layer F.SilkS) (width 0.15))
-    (fp_line (start -2.2 -0.45) (end -6.9 -0.45) (layer Dwgs.User) (width 0.15))
-    (fp_line (start -2.2 0.45) (end -2.2 -0.45) (layer Dwgs.User) (width 0.15))
-    (fp_line (start -6.9 0.45) (end -2.2 0.45) (layer Dwgs.User) (width 0.15))
-    (fp_line (start -6.9 -0.45) (end -6.9 0.45) (layer Dwgs.User) (width 0.15))
-    (fp_line (start 2.2 0.45) (end 2.2 -0.45) (layer Dwgs.User) (width 0.15))
-    (fp_line (start 6.9 0.45) (end 2.2 0.45) (layer Dwgs.User) (width 0.15))
-    (fp_line (start 6.9 -0.45) (end 6.9 0.45) (layer Dwgs.User) (width 0.15))
-    (fp_line (start 2.2 -0.45) (end 6.9 -0.45) (layer Dwgs.User) (width 0.15))
-    (fp_line (start -6.75 6.75) (end -6.75 -6.75) (layer F.SilkS) (width 0.15))
-    (fp_line (start 3.95 6.75) (end -6.75 6.75) (layer F.SilkS) (width 0.15))
-    (fp_line (start 6.75 -3.95) (end 6.75 3.95) (layer F.SilkS) (width 0.15))
-    (fp_line (start -6.75 -6.75) (end 3.95 -6.75) (layer F.SilkS) (width 0.15))
-    (fp_circle (center 0 0) (end 6.25 0) (layer F.SilkS) (width 0.15))
-    (pad 1 smd rect (at 4.55 0 90) (size 6 2.5) (layers F.Cu F.Paste F.Mask)
-      (net 1 /Vout))
-    (pad 2 smd rect (at -4.55 0 90) (size 6 2.5) (layers F.Cu F.Paste F.Mask)
-      (net 4 GND))
-  )
-  (gr_text "KIS-3R33S_breakout V0.12.d\n2015 - blog.spitzenpfeil.org" (at 157.5 107) (layer B.SilkS)
+  (gr_text "KIS-3R33S_breakout V0.12.e\n2015 - blog.spitzenpfeil.org" (at 150.5 107) (layer B.SilkS)
     (effects (font (size 1.5 1.5) (thickness 0.3)) (justify mirror))
   )
